File: PCB/psocpcb/psocpcb.kicad_pcb (KiCad board)
At the start: 2 copper layers, 66.5 x 57.5 mm, 23 parts, among them J1 Conn_01x04_Pin, J2 Conn_01x06_Pin, J3 Conn_01x04_Pin, U1 CYBLE-416045-02

Commit message: v1-review1
Parts:
- added J4: Conn_01x07_Pin, Connector_PinHeader_2.54mm:PinHeader_1x07_P2.54mm_Vertical, F.Cu at (136.8, 39.2)
Connections:
- U1 pad 26: unconnected-(U1-P6.7-Pad26) -> /SWDCLK
- U1 pad 27: unconnected-(U1-P6.6-Pad27) -> /SWDIO
- U1 pad 39: unconnected-(U1-P5.0-Pad39) -> /usbrx
- U1 pad 40: unconnected-(U1-P5.1-Pad40) -> /usbtx
Routing:
- net /XRES: track 23.9 -> 68.4 mm
- net /usbtx: track 0.00 -> 39.3 mm
- net /SWDCLK: track 0.00 -> 39.0 mm, vias 0 -> 3
- net /usbrx: track 0.00 -> 38.4 mm
- net /SWDIO: track 0.00 -> 37.2 mm, vias 0 -> 3
- net /Vdd: track 94.1 -> 125.6 mm
- net /tx: track 32.7 -> 30.4 mm, vias 2 -> 1
- net /rx: track 31.5 -> 29.6 mm, vias 2 -> 1
- net /ADC2: track 15.9 -> 17.1 mm
- net /SDA: track 63.7 -> 63.6 mm, vias 4 -> 3
- net GND: vias 7 -> 12
- net /ADC1_raw: vias 3 -> 2
Other:
- board text added: "SWDCLK"
- board text added: "SWDIO"
- board text added: "XRES"
- board text added: "dbgRX"
- board text added: "dbgTX"

Commit message: second review
Parts:
- removed C1: 0.1u, Capacitor_SMD:C_0603_1608Metric
- removed C2: 10u, Capacitor_SMD:C_0603_1608Metric
- removed J1, J3: Conn_01x04_Pin, Connector_PinHeader_2.54mm:PinHeader_1x04_P2.54mm_Vertical
- removed J2: Conn_01x06_Pin, Connector_PinHeader_2.54mm:PinHeader_1x06_P2.54mm_Vertical
- added C3: 1.0u, Capacitor_SMD:C_0603_1608Metric, B.Cu at (134.0, 50.0)
- added C4: 0.1u, Capacitor_SMD:C_0603_1608Metric, B.Cu at (152.5, 54.0)
- added C5: 1.0u, Capacitor_SMD:C_0603_1608Metric, B.Cu at (149.5, 54.0)
- added C6: 0.1u, Capacitor_SMD:C_0603_1608Metric, B.Cu at (131.0, 50.0)
- added C7: 10u, Capacitor_SMD:C_0603_1608Metric, B.Cu at (129.5, 40.5)
- added C8: 0.1u, Capacitor_SMD:C_0603_1608Metric, B.Cu at (129.5, 38.0)
- added J5: Conn_01x04_Pin, Connector_JST:JST_PH_S4B-PH-K_1x04_P2.00mm_Horizontal, F.Cu at (138.5, 82.0)
- added J6: Conn_01x04_Pin, Connector_JST:JST_PH_S4B-PH-K_1x04_P2.00mm_Horizontal, F.Cu at (126.0, 39.5)
- added J7: Conn_01x06_Pin, Connector_JST:JST_PH_S6B-PH-K_1x06_P2.00mm_Horizontal, F.Cu at (118.8, 82.0)
- R1, R10, R11, R2, R4, R6, R8: moved to B.Cu
- moved R11 24.3 mm to (106.2, 70.8)
- moved R2 22.4 mm to (131.0, 54.0), turned to 90 degrees
- moved S1 21.8 mm to (106.2, 48.8)
- moved D1 14.9 mm to (106.0, 66.5)
- moved R5 13.5 mm to (126.8, 73.2), turned to -90 degrees
- moved R9 12.6 mm to (126.8, 77.1), turned to -90 degrees
- moved R8 10.2 mm to (122.8, 77.1), turned to -90 degrees
- moved R3 6.56 mm to (120.8, 73.2), turned to -90 degrees
- moved R6 6.54 mm to (128.8, 73.2), turned to -90 degrees
- moved R7 6.24 mm to (120.8, 77.1), turned to -90 degrees
- moved R10 6.24 mm to (128.8, 77.0), turned to -90 degrees
- moved R4 5.78 mm to (122.8, 73.3), turned to -90 degrees
- moved R1 2.25 mm to (134.0, 54.0), turned to 90 degrees
Connections:
- R11 pad 2: GND -> /LED
- U1 pad 23: unconnected-(U1-P7.1-Pad23) -> /LED
Routing:
- net /Vdd: track 125.6 -> 54.8 mm, vias 4 -> 9
- net /LED: track 0.00 -> 16.7 mm, vias 0 -> 1
- net /rx: track 29.6 -> 45.6 mm, vias 1 -> 2
- net /tx: track 30.4 -> 44.9 mm, vias 1 -> 2
- net /usbtx: track 39.3 -> 53.8 mm, vias 0 -> 2
- net /usbrx: track 38.4 -> 52.8 mm, vias 0 -> 3
- net /ADC2_raw: track 17.7 -> 4.15 mm, vias 1 -> 0
- net /ADC1_raw: track 16.6 -> 4.15 mm, vias 2 -> 0
- net /ADC3_raw: track 12.7 -> 4.22 mm, vias 1 -> 0
- net /SDA: track 63.6 -> 55.5 mm
- net /ADC0_raw: track 11.2 -> 4.15 mm, vias 1 -> 0
- net /SWDIO: track 37.2 -> 43.7 mm, vias 3 -> 2
- net /XRES: track 68.4 -> 62.5 mm
- net /SWDCLK: track 39.0 -> 44.6 mm, vias 3 -> 2
- net /ADC2: track 17.1 -> 21.0 mm
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- added copper zone on B.Cu, net /Vdd
- added copper zone on F.Cu, net /Vdd
Other:
- board text added: "11/7/2024"
- board text added: "@Fall Embedded Team"
- board text added: "CMU Biorobotics Lab"
- board text added: "PAS Remote Monitoring System"
- board text added: "PSoC RPI Bottom HAT -- V1"
