File: PCB/psocpcb/psocpcb.kicad_pcb (KiCad board)
At the start: 2 copper layers, 66.5 x 57.5 mm, 28 parts, among them J4 Conn_01x07_Pin, J5 Conn_01x04_Pin, J6 Conn_01x04_Pin, J7 Conn_01x06_Pin, U1 CYBLE-416045-02

Commit message: third review
Parts:
- added D2: RED LED, LED_SMD:LED_0603_1608Metric_Pad1.05x0.95mm_HandSolder, F.Cu at (106.0, 70.7)
- added R12: 470 ohm, Resistor_SMD:R_0603_1608Metric, F.Cu at (106.0, 74.0)
Connections:
- net /LED renamed /LED1
- U1 pad 30: unconnected-(U1-P6.3-Pad30) -> /LED2
Routing:
- net /LED2: track 0.00 -> 16.6 mm
- net /Vdd: track 54.8 -> 59.0 mm
- net Net-(D2-K): track 0.00 -> 3.32 mm
- net /SWDCLK: track 44.6 -> 46.6 mm
- net /ADC3: track 22.1 -> 21.5 mm
- net /ADC1: track 22.0 -> 21.5 mm
- net GND: vias 21 -> 32
