File: PCB/psocpcb/psocpcb.kicad_sch (KiCad schematic)
At the start: 23 parts, among them J1 Conn_01x04_Pin, J2 Conn_01x06_Pin, J3 Conn_01x04_Pin, U1 CYBLE-416045-02

Commit message: v1-review1
Parts:
- added J4: Conn_01x07_Pin, Connector_PinHeader_2.54mm:PinHeader_1x07_P2.54mm_Vertical, symbol Connector:Conn_01x07_Pin
Connections:
- net GND: now also J4.6 (Pin_6)
- net Vdd: now also J4.7 (Pin_7)
- net XRES: now also J4.5 (Pin_5)
- net SWDCLK: now reaches U1.26 (P6.7)
- net SWDCLK: now also J4.4 (Pin_4)
- net SWDIO: now reaches U1.27 (P6.6)
- net SWDIO: now also J4.3 (Pin_3)
- net usbrx: now reaches U1.39 (P5.0)
- net usbrx: now also J4.1 (Pin_1)
- net usbtx: now reaches U1.40 (P5.1)
- net usbtx: now also J4.2 (Pin_2)
- no-connect marks 29 -> 25
Other:
- moved on the sheet: C1, C2, J3

Commit message: second review
Parts:
- removed C1: 0.1u, Capacitor_SMD:C_0603_1608Metric, symbol Device:C
- removed C2: 10u, Capacitor_SMD:C_0603_1608Metric, symbol Device:C
- removed J1, J3: Conn_01x04_Pin, Connector_PinHeader_2.54mm:PinHeader_1x04_P2.54mm_Vertical, symbol Connector:Conn_01x04_Pin
- removed J2: Conn_01x06_Pin, Connector_PinHeader_2.54mm:PinHeader_1x06_P2.54mm_Vertical, symbol Connector:Conn_01x06_Pin
- added C3, C5: 1.0u, Capacitor_SMD:C_0603_1608Metric, symbol Device:C
- added C4, C6, C8: 0.1u, Capacitor_SMD:C_0603_1608Metric, symbol Device:C
- added C7: 10u, Capacitor_SMD:C_0603_1608Metric, symbol Device:C
- added J5, J6: Conn_01x04_Pin, Connector_JST:JST_PH_S4B-PH-K_1x04_P2.00mm_Horizontal, symbol Connector:Conn_01x04_Pin
- added J7: Conn_01x06_Pin, Connector_JST:JST_PH_S6B-PH-K_1x06_P2.00mm_Horizontal, symbol Connector:Conn_01x06_Pin
Connections:
- net ADC0_raw: now also J7.2 (Pin_2)
- net ADC1_raw: now also J7.3 (Pin_3)
- net ADC2_raw: now also J7.5 (Pin_5)
- net ADC3_raw: now also J7.6 (Pin_6)
- net GND: now also C3.2, C4.2, C5.2, C6.2, C7.2, C8.2, J5.1 (Pin_1), J6.2 (Pin_2), J7.1 (Pin_1), J7.4 (Pin_4); no longer R11.2
- net SCL: now also J5.3 (Pin_3)
- net SDA: now also J5.4 (Pin_4)
- net Vdd: now also C3.1, C4.1, C5.1, C6.1, C7.1, C8.1, J5.2 (Pin_2), J6.1 (Pin_1)
- net rx: now also J6.4 (Pin_4)
- net tx: now also J6.3 (Pin_3)
- net LED: now reaches U1.23 (P7.1)
- net LED: now also R11.2
- no-connect marks 25 -> 24
Other:
- moved on the sheet: D1, H1, H2, H3, H4, J4, R1, R10, R11, R2, R3, R4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

Commit message: third review
Parts:
- added D2: RED LED, LED_SMD:LED_0603_1608Metric_Pad1.05x0.95mm_HandSolder, symbol Device:LED
- added R12: 470 ohm, Resistor_SMD:R_0603_1608Metric, symbol Device:R
Connections:
- net Vdd: now also D2.2 (A)
- net LED2: now reaches U1.30 (P6.3)
- net LED2: now also R12.2
- net LED renamed LED1
- new net: D2.1 (K), R12.1
- no-connect marks 24 -> 23
Other:
- moved on the sheet: J5
