File: PCB/psocpcb_v2/psocpcb.kicad_sch (KiCad schematic)
At the start: 30 parts, among them J4 Conn_01x07_Pin, J5 Conn_01x04_Pin, J6 Conn_01x04_Pin, J7 Conn_01x06_Pin, U1 CYBLE-416045-02

Commit message: schematic
Parts:
- removed D1: Green LED, LED_SMD:LED_0603_1608Metric_Pad1.05x0.95mm_HandSolder, symbol Device:LED
- removed D2: RED LED, LED_SMD:LED_0603_1608Metric_Pad1.05x0.95mm_HandSolder, symbol Device:LED
- removed H1, H2, H3, H4: MountingHole, MountingHole:MountingHole_2.7mm_M2.5_Pad_TopBottom, symbol Mechanical:MountingHole
- removed J4: Conn_01x07_Pin, Connector_PinHeader_2.54mm:PinHeader_1x07_P2.54mm_Vertical, symbol Connector:Conn_01x07_Pin
- removed J6: Conn_01x04_Pin, Connector_JST:JST_PH_S4B-PH-K_1x04_P2.00mm_Horizontal, symbol Connector:Conn_01x04_Pin
- removed S1: SKRPACE010, kicad library:SW_SKRPACE010, symbol SKswitch:SKRPACE010
- removed U1: CYBLE-416045-02, kicad library:XCVR_CYBLE-416045-02, symbol CYBLE-416045-02:CYBLE-416045-02
- added A1: RASPBERRYPI-ZERO, RASPBERRYPI-ZERO:RASPBERRYPI-ZERO_RPI-ZERO, symbol RASPBERRYPI-ZERO:RASPBERRYPI-ZERO
- added C1, C2: 22pF, Capacitor_SMD:C_0603_1608Metric, symbol Device:C
- added C10, C12, C17, C19: 4.7uF, Capacitor_SMD:C_0603_1608Metric, symbol Device:C
- added C11, C18, C9: 0.1uF, Capacitor_SMD:C_0603_1608Metric, symbol Device:C
- added C13, C14: 0.1u, Capacitor_SMD:C_0603_1608Metric, symbol Device:C
- added D1, D2: LTST-C190CKT, LTST-C190CKT:LEDSC160X80X90-2N, symbol LTST-C190CKT:LTST-C190CKT
- added FB1: FerriteBead, Inductor_SMD:L_0603_1608Metric, symbol Device:FerriteBead
- added J1: Conn_01x05, Connector_PinHeader_2.54mm:PinHeader_1x05_P2.54mm_Horizontal, symbol Connector_Generic:Conn_01x05
- added J2: Conn_01x02_Pin, Connector_PinHeader_2.54mm:PinHeader_1x02_P2.54mm_Vertical, symbol Connector:Conn_01x02_Pin
- added Q1: Si2337DS, Package_TO_SOT_SMD:SOT-23, symbol Transistor_FET:AO3401A
- added R13: 180K, Resistor_SMD:R_0603_1608Metric, symbol Device:R
- added R14: 57.6K, Resistor_SMD:R_0603_1608Metric, symbol Device:R
- added R15: 200K, Resistor_SMD:R_0603_1608Metric, symbol Device:R
- added R16: 160K, Resistor_SMD:R_0603_1608Metric, symbol Device:R
- added U2, U6: AP7365-WG-7, AP7365-33WG-7:SOT95P285X145-5N, symbol Regulator_Linear:LDK130-ADJ_SOT23_SOT353
- added U3: AP2331SA-7, AP2331SA-7:SOT91P240X120-3N, symbol AP2331SA-7:AP2331SA-7
- added U4: SIP32408DNP-T1-GE4, SIP32408DNP-T1-GE4:SON50P120X160X60-5N, symbol SIP32408DNP-T1-GE4:SIP32408DNP-T1-GE4
- added U5: TXS0102DCUR, TXS0102DCUR:SOP50P310X90-8N, symbol TXS0102DCUR:TXS0102DCUR
- added U7: CYBLE-416045-02, CYBLE-416045-02:XCVR_CYBLE-416045-02, symbol CYBLE-416045-02:CYBLE-416045-02
- added Y1: ECS-.327-12.5-34B-TR, ECS-.327-12.5-34B-TR:XTAL_ECS-.327-12.5-34B-TR, symbol ECS-.327-12.5-34B-TR:ECS-.327-12.5-34B-TR
- C7: value 10u -> 0.1u
- R10, R7, R8, R9: value 18k -> 20K
- R11: value 330 ohm -> ~
- R3, R4, R5, R6: value 6.8k -> 10K
Connections:
- net LED2 is gone; now on net LED1: R12.2
- net ADC0: now also C7.2, U7.7 (P10.3)
- net ADC1: now also C8.2, U7.8 (P10.4)
- net ADC2: now also C13.2, U7.11 (P10.5)
- net ADC3: now also C14.2, U7.10 (P10.6)
- net GND: now also R11.2, A1.14 (GND[4]), A1.20 (GND[5]), A1.25 (GND[2]), A1.30 (GND[6]), A1.34 (GND[7]), A1.39 (GND[3]), A1.6 (GND[8]), A1.9 (GND[1]), C1.2, C10.2, C11.2, C12.2, C17.2, C18.2, C19.2, C2.2, C9.2, FB1.1, J1.4 (Pin_4), R14.2, R16.2, U2.2 (GND), U3.1 (GND), U4.2 (GND), U4.5 (GND), U5.2 (GND), U6.2 (GND), U7.1 (GND), U7.15 (GND), U7.43 (GND); no longer C7.2, C8.2, J7.1 (Pin_1), J7.4 (Pin_4), R3.1, R4.1, R5.1, R6.1
- net LED1: now also U7.30 (P6.3); no longer R11.2
- net SCL: now also U5.1 (B2), U7.12 (P10.1); no longer J5.3 (Pin_3)
- net SDA: now also U5.8 (B1), U7.33 (P10.2); no longer J5.4 (Pin_4)
- net SWDCLK: now also J1.2 (Pin_2), U7.26 (P6.7)
- net SWDIO: now also J1.1 (Pin_1), U7.27 (P6.6)
- net XRES: now also J1.3 (Pin_3), U7.42 (XRES)
- net usbrx: now also J2.2 (Pin_2), U7.39 (P5.0)
- net usbtx: now also J2.1 (Pin_1), U7.40 (P5.1)
- net at R11.1: now also D2.C
- net at R12.1: now also D1.C
- net Vdd renamed VTAG
- net VTAG: now also C17.1, C18.1, D1.A, J1.5 (Pin_5), U4.4 (OUT), U5.7 (VCCB), U6.1 (IN), U6.3 (EN), U7.3 (VBACKUP), U7.4 (VDD); no longer C7.1, C8.1, J5.2 (Pin_2)
- new net: C2.1, U7.5 (P0.0), Y1.2
- new net: A1.2 (5V[1]), A1.4 (5V[2]), Q1.2 (S)
- new net: C1.1, U7.6 (P0.1), Y1.1
- new net: R13.2, R14.1, U2.4 (ADJ)
- new net: R15.2, R16.1, U6.4 (ADJ)
- new net 1.8V: C19.1, R15.1, U5.3 (VCCA), U5.6 (OE), U6.5 (OUT)
- new net 5V: C10.1, C11.1, C9.1, D2.A, J5.2 (Pin_2), U2.1 (IN), U2.3 (EN), U3.2 (OUT)
- new net 5V_IN: Q1.3 (D), U3.3 (IN)
- new net GNDA: C13.1, C14.1, C7.1, C8.1, FB1.2, J7.1 (Pin_1), J7.4 (Pin_4), R3.1, R4.1, R5.1, R6.1
- new net MCURX: A1.8 (TXD0/GPIO14), U7.17 (P9.0)
- new net MCUTX: A1.10 (RXD0/GPIO15), U7.18 (P9.1)
- new net SCL1.8: J5.3 (Pin_3), U5.4 (A2)
- new net SDA1.8: J5.4 (Pin_4), U5.5 (A1)
- new net VOUT: C12.1, R13.1, U2.5 (OUT), U4.1 (IN), U4.3 (EN)
- new net reset: A1.7 (GPIO4/GPCKL0), Q1.1 (G)
- no-connect marks 23 -> 49
Other:
- company: (none) -> Carnegie Mellon University Biorobotics Lab
- title: (none) -> ECMOPCBv2
- moved on the sheet: C3, C4, C5, C6, J5, J7, R1, R11, R12, R2, R3, R7

Commit message: pulldown
Parts:
- added R17: 4.7K, Resistor_SMD:R_0603_1608Metric, symbol Device:R
Connections:
- net GND: now also R17.1
- net reset: now also R17.2
Changed lines of the file:
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@@
 	(wire
 		(pts
-			(xy 264.16 38.1) (xy 273.05 38.1)
-		)
-		(stroke
-			(width 0)
-			(type default)
-		)
-	)
-	(wire
-		(pts
 			(xy 63.5 36.83) (xy 48.26 36.83)
 		)
@@
 	(wire
 		(pts
+			(xy 264.16 38.1) (xy 264.16 39.37)
+		)
+		(stroke
+			(width 0)
+			(type default)
+		)
+	)
+	(wire
+		(pts
 			(xy 176.53 72.39) (xy 186.69 72.39)
 		)
@@
 	(wire
 		(pts
+			(xy 264.16 38.1) (xy 273.05 38.1)
+		)
+		(stroke
+			(width 0)
+			(type default)
+		)
+	)
+	(wire
+		(pts
 			(xy 105.41 184.15) (xy 111.76 184.15)
 		)
@@
 	)
 	(symbol
+		(lib_id "Device:R")
+		(at 264.16 43.18 0)
+		(mirror x)
+		(unit 1)
+		(exclude_from_sim no)
+		(in_bom yes)
+		(on_board yes)
+		(dnp no)
+		(property "Reference" "R17"
+			(at 261.62 41.9099 0)
+			(effects
+				(font
+					(size 1.27 1.27)
+				)
+				(justify right)
+			)
+		)
+		(property "Value" "4.7K"
+			(at 261.62 44.4499 0)
+			(effects
+				(font
+					(size 1.27 1.27)
+				)
+				(justify right)
+			)
+		)
+		(property "Footprint" "Resistor_SMD:R_0603_1608Metric"
+			(at 262.382 43.18 90)
+			(effects
+				(font
+					(size 1.27 1.27)
+				)
+				(hide yes)
+			)
+		)
+		(property "Datasheet" "~"
+			(at 264.16 43.18 0)
+			(effects
+				(font
+					(size 1.27 1.27)
+				)
+				(hide yes)
+			)
+		)
+		(property "Description" "Resistor"
+			(at 264.16 43.18 0)
+			(effects
+				(font
+					(size 1.27 1.27)
+				)
+				(hide yes)
+			)
+		)
+		(pin "1"
+		)
+		(pin "2"
+		)
+		(instances
+			(project "psocpcb"
+				(path "/b99eb613-5e3f-4ea6-a2aa-d7f60f888a4d"
+					(reference "R17")
+					(unit 1)
+				)
+			)
+		)
+	)
+	(symbol
 		(lib_id "Device:C")
 		(at 140.97 30.48 0)
@@
 					(unit 1)
 				)
+			)
+		)
+	)
+	(symbol
+		(lib_id "power:GND")
+		(at 264.16 46.99 0)
+		(unit 1)
+		(exclude_from_sim no)
+		(in_bom yes)
+		(on_board yes)
+		(dnp no)
+		(fields_autoplaced yes)
+		(property "Reference" "#PWR044"
+			(at 264.16 53.34 0)
+			(effects
+				(font
+					(size 1.27 1.27)
+				)
+				(hide yes)
+			)
+		)
+		(property "Value" "GND"
+			(at 264.16 52.07 0)
+			(effects
+				(font
+					(size 1.27 1.27)
+				)
+			)
+		)
+		(property "Footprint" ""
+			(at 264.16 46.99 0)
+			(effects
+				(font
+					(size 1.27 1.27)
+				)
+				(hide yes)
+			)
+		)
+		(property "Datasheet" ""
+			(at 264.16 46.99 0)
+			(effects
+				(font
+					(size 1.27 1.27)
+				)
+				(hide yes)
+			)
+		)
+		(property "Description" "Power symbol creates a global label with name \"GND\" , ground"
+			(at 264.16 46.99 0)
+			(effects
+				(font
+					(size 1.27 1.27)
+				)
+				(hide yes)
+			)
+		)
+		(pin "1"
+		)
+		(instances
+			(project "psocpcb"
+				(path "/b99eb613-5e3f-4ea6-a2aa-d7f60f888a4d"
+					(reference "#PWR044")
+					(unit 1)
+				)

Commit message: L1
Parts:
- A1: footprint RASPBERRYPI-ZERO:RASPBERRYPI-ZERO_RPI-ZERO -> RASPBERRYPI-ZERO:RASPBERRYPI-ZERO_RPI-ZERO_1
- J1: footprint Connector_PinHeader_2.54mm:PinHeader_1x05_P2.54mm_Horizontal -> Connector_PinHeader_2.54mm:PinHeader_1x05_P2.54mm_Vertical
Connections:
- net ADC0_raw: now also J7.6 (Pin_6); no longer J7.2 (Pin_2)
- net ADC1_raw: now also J7.5 (Pin_5); no longer J7.3 (Pin_3)
- net ADC2_raw: now also J7.2 (Pin_2); no longer J7.5 (Pin_5)
- net ADC3_raw: now also J7.3 (Pin_3); no longer J7.6 (Pin_6)
- net GND: now also C13.1, C14.1, C7.1, C8.1
- net GNDA: no longer C13.1, C14.1, C7.1, C8.1

Commit message: layout Finished
Parts:
- removed C6: 0.1u, Capacitor_SMD:C_0603_1608Metric, symbol Device:C
- C5: value 1.0u -> 10u
Changed lines of the file:
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@@
 	)
 	(junction
-		(at 140.97 21.59)
-		(diameter 0)
-		(color 0 0 0 0)
-	)
-	(junction
 		(at 78.74 115.57)
 		(diameter 0)
@@
 	(wire
 		(pts
-			(xy 152.4 21.59) (xy 152.4 26.67)
-		)
-		(stroke
-			(width 0)
-			(type default)
-		)
-	)
-	(wire
-		(pts
 			(xy 58.42 184.15) (xy 68.58 184.15)
 		)
@@
 	(wire
 		(pts
-			(xy 140.97 21.59) (xy 152.4 21.59)
-		)
-		(stroke
-			(width 0)
-			(type default)
-		)
-	)
-	(wire
-		(pts
 			(xy 140.97 21.59) (xy 140.97 26.67)
 		)
@@
 			)
 		)
-		(property "Value" "1.0u"
+		(property "Value" "10u"
 			(at 144.78 31.7499 0)
 			(effects
@@
 	)
 	(symbol
-		(lib_id "power:GND")
-		(at 152.4 34.29 0)
-		(unit 1)
-		(exclude_from_sim no)
-		(in_bom yes)
-		(on_board yes)
-		(dnp no)
-		(fields_autoplaced yes)
-		(property "Reference" "#PWR017"
-			(at 152.4 40.64 0)
-			(effects
-				(font
-					(size 1.27 1.27)
-				)
-				(hide yes)
-			)
-		)
-		(property "Value" "GND"
-			(at 152.4 39.37 0)
-			(effects
-				(font
-					(size 1.27 1.27)
-				)
-			)
-		)
-		(property "Footprint" ""
-			(at 152.4 34.29 0)
-			(effects
-				(font
-					(size 1.27 1.27)
-				)
-				(hide yes)
-			)
-		)
-		(property "Datasheet" ""
-			(at 152.4 34.29 0)
-			(effects
-				(font
-					(size 1.27 1.27)
-				)
-				(hide yes)
-			)
-		)
-		(property "Description" "Power symbol creates a global label with name \"GND\" , ground"
-			(at 152.4 34.29 0)
-			(effects
-				(font
-					(size 1.27 1.27)
-				)
-				(hide yes)
-			)
-		)
-		(pin "1"
-		)
-		(instances
-			(project "psocpcb"
-				(path "/b99eb613-5e3f-4ea6-a2aa-d7f60f888a4d"
-					(reference "#PWR017")
-					(unit 1)
-				)
-			)
-		)
-	)
-	(symbol
 		(lib_id "power:GNDA")
 		(at 20.32 162.56 0)
@@
 					(unit 1)
 				)
-			)
-		)
-	)
-	(symbol
-		(lib_id "Device:C")
-		(at 152.4 30.48 0)
-		(unit 1)
-		(exclude_from_sim no)
-		(in_bom yes)
-		(on_board yes)
-		(dnp no)
-		(fields_autoplaced yes)
-		(property "Reference" "C6"
-			(at 156.21 29.2099 0)
-			(effects
-				(font
-					(size 1.27 1.27)
-				)
-				(justify left)
-			)
-		)
-		(property "Value" "0.1u"
-			(at 156.21 31.7499 0)
-			(effects
-				(font
-					(size 1.27 1.27)
-				)
-				(justify left)
-			)
-		)
-		(property "Footprint" "Capacitor_SMD:C_0603_1608Metric"
-			(at 153.3652 34.29 0)
-			(effects
-				(font
-					(size 1.27 1.27)
-				)
-				(hide yes)
-			)
-		)
-		(property "Datasheet" "~"
-			(at 152.4 30.48 0)
-			(effects
-				(font
-					(size 1.27 1.27)
-				)
-				(hide yes)
-			)
-		)
-		(property "Description" "Unpolarized capacitor"
-			(at 152.4 30.48 0)
-			(effects
-				(font
-					(size 1.27 1.27)
-				)
-				(hide yes)
-			)
-		)
-		(pin "1"
-		)
-		(pin "2"
-		)
-		(instances
-			(project "psocpcb"
-				(path "/b99eb613-5e3f-4ea6-a2aa-d7f60f888a4d"
-					(reference "C6")
-					(unit 1)
-				)
