File: PCB/psocpcb_v2/psocpcb.kicad_sch (KiCad schematic)
At the start: 49 parts, among them J1 Conn_01x05, J2 Conn_01x02_Pin, J5 Conn_01x04_Pin, J7 Conn_01x06_Pin, Q1 Si2337DS, U2 AP7365-WG-7, U3 AP2331SA-7, U4 SIP32408DNP-T1-GE4, U5 TXS0102DCUR, U6 AP7365-WG-7, U7 CYBLE-416045-02, Y1 ECS-.327-12.5-34B-TR

Commit message: Minor Revise
Parts:
- U7: footprint CYBLE-416045-02:XCVR_CYBLE-416045-02 -> RASPBERRYPI-ZERO:RASPBERRYPI-ZERO_RPI-ZERO_1_1
Changed lines of the file:
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@@
 			)
 		)
-		(property "Footprint" "CYBLE-416045-02:XCVR_CYBLE-416045-02"
+		(property "Footprint" "RASPBERRYPI-ZERO:RASPBERRYPI-ZERO_RPI-ZERO_1_1"
 			(at 83.82 57.15 0)
 			(effects
